File: pcb/Untitled.kicad_pcb (KiCad board)
At the start: 2 copper layers, 91.5 x 100 mm, 57 parts, among them J1 Conn_01x08_Socket, J2 Micro_SD_Card_Det1, J3 USB_C_Receptacle_USB2.0_14P, J4 Conn_01x02, J5 Conn_Coaxial, Q1 FS8205A, Q2 AO3407A, SW1 reset, SW10 SW_Push, SW2 boot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

Commit message: update
Parts:
- removed C3: 0.1uF, Capacitor_SMD:C_0402_1005Metric
- removed U7: LIS3MDL, Package_LGA:LGA-12_2x2mm_P0.5mm
- added C8: 220nF, Capacitor_SMD:C_0402_1005Metric, F.Cu at (174.3, 78.8)
- added U8: LIS2MDL, Package_LGA:LGA-12_2x2mm_P0.5mm, F.Cu at (174.5, 80.5)
- Q1: footprint FS8205A:SOP65P640X120-8N -> Package_TO_SOT_SMD:SOT-23-6
- moved D1 12.6 mm to (246.0, 34.2)
- moved R5 9.74 mm to (247.7, 36.5), turned to 180 degrees
- moved SW4 9.25 mm to (213.8, 54.8)
- moved SW3 7.25 mm to (213.8, 47.5)
- moved SW9 4.50 mm to (232.2, 115.0)
- moved SW6 4.25 mm to (228.5, 57.0)
- moved SW10 3.64 mm to (247.8, 100.5)
- moved SW8 3.64 mm to (216.8, 100.5)
- moved SW5 2.57 mm to (244.0, 66.5)
- moved SW7 2.50 mm to (232.2, 86.0)
- moved Q1 1.82 mm to (186.2, 60.0), turned to -90 degrees
- moved J1 0.75 mm to (182.0, 112.2)
Routing:
- net Net-(U2-TIMEPULSE): track 2.28 -> 12.0 mm
- net IO39: track 34.1 -> 43.2 mm
- net IO40: track 43.6 -> 49.7 mm
- net GND: track 99.2 -> 94.0 mm, vias 17 -> 16
- net IO47: track 51.2 -> 46.7 mm
- net IO42: track 48.1 -> 52.4 mm
- net SDA: track 36.9 -> 33.0 mm
- net IO09: track 47.5 -> 51.3 mm
- net IO21: track 24.0 -> 20.9 mm
- net IO48: track 49.5 -> 47.0 mm
- net SCL: track 38.6 -> 36.2 mm
- net IO41: track 43.8 -> 46.0 mm
- net Net-(U6-OD): track 6.48 -> 4.54 mm
- net BAT-: track 22.8 -> 24.7 mm
- net Net-(U1-IO0): track 65.4 -> 63.6 mm
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