File: pcb/Untitled.kicad_pcb (KiCad board)
At the start: 2 copper layers, 91.5 x 100 mm, 57 parts, among them J1 Conn_01x08_Socket, J2 Micro_SD_Card_Det1, J3 USB_C_Receptacle_USB2.0_14P, J4 Conn_01x02, J5 Conn_Coaxial, Q1 FS8205A, Q2 AO3407A, SW1 reset, SW10 SW_Push, SW2 boot, SW3 SW_Push, SW4 SW_Push, SW5 SW_Push, SW6 SW_Push, SW7 SW_Push, SW8 SW_Push, SW9 SW_Push, U1 ESP32-S3-WROOM-1, U10 RV-3028-C8-32.768KHZ-1PPM-TA-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, U11 BMP390, U2 MAX-M10S, U3 USBLC6-2SC6, U4 MCP73831-2-MC, U5 AP2112K-3.3, U6 DW01A, U8 LIS2MDL, U9 SHT4x

Commit message: update
Parts:
- moved C8 15.2 mm to (174.3, 94.0)
- moved U8 15.2 mm to (174.5, 95.8)
- moved R5 0.51 mm to (247.6, 37.0)
- moved D1 0.51 mm to (245.9, 34.8)
- moved J1 0.35 mm to (181.7, 112.2)
Routing:
- net SDA: track 33.0 -> 42.4 mm
- net +3V3: track 244.9 -> 252.8 mm
- net SCL: track 36.2 -> 40.0 mm
- net IO13: track 105.6 -> 108.8 mm
- net IO47: track 46.7 -> 47.3 mm
- net IO09: track 51.3 -> 51.9 mm
Other:
- board text added: "by kate"
- board text added: "made with"
