File: pcb/Untitled.kicad_pcb (KiCad board)
At the start: 2 copper layers, 91.5 x 100 mm, 57 parts, among them J1 Conn_01x08_Socket, J2 Micro_SD_Card_Det1, J3 USB_C_Receptacle_USB2.0_14P, J4 Conn_01x02, J5 Conn_Coaxial, Q1 FS8205A, Q2 AO3407A, SW1 reset, SW10 SW_Push, SW2 boot, SW3 SW_Push, SW4 SW_Push, SW5 SW_Push, SW6 SW_Push, SW7 SW_Push, SW8 SW_Push, SW9 SW_Push, U1 ESP32-S3-WROOM-1, U10 RV-3028-C8-32.768KHZ-1PPM-TA-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, U11 BMP390, U2 MAX-M10S, U3 USBLC6-2SC6, U4 MCP73831-2-MC, U5 AP2112K-3.3, U6 DW01A, U8 LIS2MDL, U9 SHT4x

Commit message: update
Parts:
- removed C6: 0.1uF, Capacitor_SMD:C_0402_1005Metric
- removed U10: RV-3028-C8-32.768KHZ-1PPM-TA-QC, footprintsrv:IC_RV-3028-C8-32.768KHZ-1PPM-TA-QC
- added C14: 0.1uF, Capacitor_SMD:C_0402_1005Metric, F.Cu at (190.7, 80.6)
- added U7: RV-3028-C7, Package_SON:MicroCrystal_C7_SON-8_1.5x3.2mm_P0.9mm, F.Cu at (192.6, 81.2)
Routing:
- net SCL: track 40.0 -> 35.3 mm
- net SDA: track 42.4 -> 38.4 mm
