File: pcb/Untitled.kicad_sch (KiCad schematic)
At the start: 56 parts, among them J1 Conn_01x09, J2 Micro_SD_Card_Det1, J3 USB_C_Receptacle_USB2.0_14P, J4 Conn_01x02, J5 Conn_Coaxial, Q1 FS8205A, Q2 AO3407A, SW1 reset, SW10 SW_Push, SW2 boot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

Commit message: schematic
Parts:
- removed C8: 100nF, symbol Device:C
- removed J1: Conn_01x09, symbol Connector_Generic:Conn_01x09
- removed U8: BMP390, BMP390:BMP390, symbol BMP390:BMP390
- added C12, C13: 0.1UF, Capacitor_SMD:C_0402_1005Metric, symbol Device:C
- added J1: Conn_01x08_Socket, Connector_PinSocket_2.54mm:PinSocket_1x08_P2.54mm_Horizontal, symbol Connector:Conn_01x08_Socket
- added U11: BMP390, footprints:10LGA_2X2X0p75_BOS, symbol 2026-06-26_15-33-47:BMP390
- C1, C10, C11, C2, C4: footprint (none) -> Capacitor_SMD:C_0402_1005Metric
- C3, C6, C7, C9: value 100nF -> 0.1uF; footprint (none) -> Capacitor_SMD:C_0402_1005Metric
- C5: footprint (none) -> Capacitor_SMD:C_0603_1608Metric
- D1, D3: footprint (none) -> LED_SMD:LED_1210_3225Metric
- J2: footprint (none) -> Connector_Card:microSD_HC_Hirose_DM3AT-SF-PEJM5
- J3: footprint (none) -> Connector_USB:USB_C_Receptacle_HRO_TYPE-C-31-M-12
- J4: footprint (none) -> Connector_JST:JST_PH_S2B-PH-K_1x02_P2.00mm_Horizontal
- J5: footprint (none) -> Connector_Coaxial:SMA_Amphenol_132289_EdgeMount
- L1: value 56nH -> 27nH; footprint (none) -> Inductor_SMD:L_0402_1005Metric
- R1, R10, R11, R12, R13, R2, R3, R4, R5, R6, R7, R8, R9: footprint (none) -> Resistor_SMD:R_0402_1005Metric
- R14: value 10k -> 2k; footprint (none) -> Resistor_SMD:R_0402_1005Metric
- SW1, SW2, SW3, SW4: footprint (none) -> Button_Switch_THT:SW_TH_Tactile_Omron_B3F-100x
- SW10, SW5, SW6, SW7, SW8, SW9: footprint (none) -> Button_Switch_THT:SW_SPST_Omron_B3F-40xx
- U1: footprint RF_Module:ESP32-S3-WROOM-1 -> RF_Module:ESP32-S3-WROOM-1U
- U10: footprint RV-3028-C8-32.768KHZ-1PPM-TA-QC:IC_RV-3028-C8-32.768KHZ-1PPM-TA-QC -> footprintsrv:IC_RV-3028-C8-32.768KHZ-1PPM-TA-QC
- U4: footprint Package_DFN_QFN:DFN-8-1EP_3x2mm_P0.5mm_EP1.7x1.4mm -> Package_TO_SOT_SMD:SOT-23-5
Connections:
- net +3V3: now also C12.1, C13.1, U11.6 (CSB)
- net +5V: now also U4.4 (V_{BAT}); no longer U4.1 (V_{DD}), U4.2 (V_{DD})
- net GND: now also U4.2 (V_{SS}), J1.2 (Pin_2), U11.3 (VSS), U11.5 (SDO), U11.8 (VSS), U11.9 (VSS); no longer U4.6 (V_{SS})
- net IO06: now also J1.5 (Pin_5)
- net IO07: now also J1.6 (Pin_6)
- net IO08: now also J1.7 (Pin_7)
- net IO09: now also J1.8 (Pin_8)
- net IO11: now also J1.3 (Pin_3)
- net IO12: now also J1.4 (Pin_4)
- net IO15: now also U4.1 (STAT); no longer U4.5 (STAT)
- net SCL: now also U11.2 (SCK)
- net SDA: now also U11.4 (SDI)
- net at R10.1: now also U4.5 (PROG); no longer U4.8 (PROG)
- net at Q2.3: now also J1.1 (Pin_1)
- new net: C13.2, U11.1 (VDDIO)
- new net: C12.2, U11.10 (VDD)

Commit message: update
Parts:
- removed C3: 0.1uF, Capacitor_SMD:C_0402_1005Metric, symbol Device:C
- removed U7: LIS3MDL, Package_LGA:LGA-12_2x2mm_P0.5mm, symbol Sensor_Magnetic:LIS3MDL
- added C8: 220nF, Capacitor_SMD:C_0402_1005Metric, symbol Device:C
- added U8: LIS2MDL, Package_LGA:LGA-12_2x2mm_P0.5mm, symbol Sensor_Magnetic:LIS2MDL
- Q1: footprint FS8205A:SOP65P640X120-8N -> Package_TO_SOT_SMD:SOT-23-6
Connections:
- net +3V3: now also U8.10 (Vdd_IO), U8.3 (~{CS}), U8.9 (Vdd)
- net GND: now also C8.2, U8.6 (GND), U8.8 (GND)
- net SCL: now also U8.1 (SCL/SPC)
- net SDA: now also U8.4 (SDA/SDI/SDO)
- new net: C8.1, U8.5 (C1)
- no-connect marks 24 -> 23
